File: pcb/charger.sch (KiCad schematic (older format))
At the start: 12 parts

Commit message: nightly | pcb build, routing, placing
Parts:
- added R501: 0R0, Resistors_SMD:R_0603_HandSoldering, symbol R
- added R502: N/A, Resistors_SMD:R_0603_HandSoldering, symbol R
- added TP501: temp, Measurement_Points:Measurement_Point_Round-SMD-Pad_Big, symbol TEST
- added TP502: Charge, Measurement_Points:Measurement_Point_Round-SMD-Pad_Big, symbol TEST
- added TP503: Standby, Measurement_Points:Measurement_Point_Round-SMD-Pad_Big, symbol TEST
- C501: renamed from C?; footprint (none) -> Capacitors_SMD:C_0603_HandSoldering
- C502: renamed from C?; footprint (none) -> Capacitors_SMD:C_1210_HandSoldering
- R503, R504, R505, R506, R509, R510, R511: renamed from R?; footprint (none) -> Resistors_SMD:R_0603_HandSoldering
- R507: renamed from R?; value 0R0 -> n/a; footprint (none) -> Resistors_SMD:R_0603_HandSoldering
- R508: renamed from R?; value N/A -> 0R0; footprint (none) -> Resistors_SMD:R_0603_HandSoldering
- U501: renamed from U?; footprint (none) -> footprints:SOP-8
Connections:
- net labels added: +5VD, -BATT
- net labels removed: DISABLE_CHARGE
- wire segments 41 -> 51
Other:
- moved on the sheet: C501
